File: 9k-mania-macropad/schematic/mania-macropad-schematic/mania-macropad-schematic.kicad_pcb (KiCad board)
At the start: 4 copper layers, 225 x 125 mm, 86 parts, among them SW1 SW_Push, U1 SW_MX_HE, U10 SW_MX_HE, U11 SW_MX_HE, U2 SW_MX_HE, U3 SW_MX_HE, U4 SW_MX_HE, U5 SW_MX_HE, U6 Teensy4.0, U7 SW_MX_HE, U8 SW_MX_HE, U9 SW_MX_HE

Commit message: Attempt to fix PCB at school
Parts:
- moved U2 0.58 mm to (72.4, 72.5)
- moved U3 0.58 mm to (91.5, 72.5)
- moved U1 0.58 mm to (53.4, 72.5)
- moved U4 0.58 mm to (110.5, 72.5)
- moved U10 0.38 mm to (219.4, 72.5)
- moved U11 0.38 mm to (238.5, 72.5)
- moved U8 0.38 mm to (181.3, 72.5)
- moved U9 0.38 mm to (200.4, 72.5)
- moved U5 0.15 mm to (98.3, 129.7)
